File: old/GuitarBot_Solenoid_Driver_PCB.kicad_sch (KiCad schematic)
At the start: 30 parts, among them J1 Screw_Terminal_01x02, J2 Screw_Terminal_01x16, J3 Screw_Terminal_01x16, J4 Screw_Terminal_01x04, SW1 SW_DIP_x03, U1 MCP23017_SP, U2 ULN2803A, U3 ULN2803A

Commit message: Modified ./old schematic to use NMOS instead of Darlington transistor array
Parts:
- removed D1, D10, D11, D12, D13, D14, D15, D16, D2, D3, D4, D5, D6, D7, D8, D9: 1N4001, Diode_SMD:D_0402_1005Metric, symbol Diode:1N4001
- removed SW1: SW_DIP_x03, Button_Switch_THT:SW_DIP_SPSTx03_Slide_9.78x9.8mm_W7.62mm_P2.54mm, symbol Switch:SW_DIP_x03
- removed U2, U3: ULN2803A, Package_SO:SOIC-18W_7.5x11.6mm_P1.27mm, symbol Transistor_Array:ULN2803A
- added D1, D10, D11, D12, D13, D14, D15, D16, D2, D3, D4, D5, D6, D7, D8, D9: D_Schottky, symbol Device:D_Schottky
- added JP1, JP2, JP3: SolderJumper_2_Open, symbol Jumper:SolderJumper_2_Open
- added Q1, Q10, Q11, Q12, Q13, Q14, Q15, Q16, Q2, Q3, Q4, Q5, Q6, Q7, Q8, Q9: NMOS, symbol Simulation_SPICE:NMOS
Connections:
- net +12V: now also D1.1 (K), D10.1 (K), D11.1 (K), D12.1 (K), D13.1 (K), D14.1 (K), D15.1 (K), D16.1 (K), D2.1 (K), D3.1 (K), D4.1 (K), D5.1 (K), D6.1 (K), D7.1 (K), D8.1 (K), D9.1 (K)
- net +3.3V: now also JP1.1 (A), JP2.1 (A), JP3.1 (A)
- net GNDPWR: now also Q1.3 (S), Q10.3 (S), Q11.3 (S), Q12.3 (S), Q13.3 (S), Q14.3 (S), Q15.3 (S), Q16.3 (S), Q2.3 (S), Q3.3 (S), Q4.3 (S), Q5.3 (S), Q6.3 (S), Q7.3 (S), Q8.3 (S), Q9.3 (S)
- net Sol1: now also Q1.2 (G)
- net Sol10: now also Q10.2 (G)
- net Sol11: now also Q11.2 (G)
- net Sol12: now also Q12.2 (G)
- net Sol13: now also Q13.2 (G)
- net Sol14: now also Q14.2 (G)
- net Sol15: now also Q15.2 (G)
- net Sol16: now also Q16.2 (G)
- net Sol2: now also Q2.2 (G)
- net Sol3: now also Q3.2 (G)
- net Sol4: now also Q4.2 (G)
- net Sol5: now also Q5.2 (G)
- net Sol6: now also Q6.2 (G)
- net Sol7: now also Q7.2 (G)
- net Sol8: now also Q8.2 (G)
- net Sol9: now also Q9.2 (G)
- net at J2.15 (Pin_15): now also D15.2 (A), Q15.1 (D)
- net at J2.16 (Pin_16): now also D16.2 (A), Q16.1 (D)
- net at J2.8 (Pin_8): now also D8.2 (A), Q1.1 (D)
- net at J2.7 (Pin_7): now also D7.2 (A), Q2.1 (D)
- net at J2.6 (Pin_6): now also D6.2 (A), Q3.1 (D)
- net at J2.5 (Pin_5): now also D5.2 (A), Q4.1 (D)
- net at J2.4 (Pin_4): now also D4.2 (A), Q5.1 (D)
- net at J2.3 (Pin_3): now also D3.2 (A), Q6.1 (D)
- net at J2.2 (Pin_2): now also D2.2 (A), Q7.1 (D)
- net at J2.1 (Pin_1): now also D1.2 (A), Q8.1 (D)
- net at J2.14 (Pin_14): now also D14.2 (A), Q14.1 (D)
- net at R5.1, U1.17 (A2): now also JP3.2 (B)
- net at R3.1, U1.15 (A0): now also JP1.2 (B)
- net at J2.11 (Pin_11): now also D11.2 (A), Q11.1 (D)
- net at R4.1, U1.16 (A1): now also JP2.2 (B)
- net at J2.9 (Pin_9): now also D9.2 (A), Q9.1 (D)
- net at J2.10 (Pin_10): now also D10.2 (A), Q10.1 (D)
- net at J2.12 (Pin_12): now also D12.2 (A), Q12.1 (D)
- net at J2.13 (Pin_13): now also D13.2 (A), Q13.1 (D)
Other:
- moved on the sheet: C1, J1, J2, J3, J4, R1, R2, R3, R4, R5, U1
